Commit message: fix: sim 验证套件——ring time 字段（微秒）/轮向轴修复/office 南墙/评测进程卫生与时间戳/轮半径标定
- ring_fill_node 补 time(float32, 微秒) 字段：与 Velodyne 预处理(×1e-3→ms, /1000→s) 单位链一致，
  消除 "Failed to find match for field 'time'"（LIO 冻结根因之一）
- adapt_urdf 轮关节轴 0 -1 0 → 0 1 0：正轮速前向（+cmd_vel → GT x 增加），/odom_wheel 与
  diff_drive odom 符号与真实运动一致（WheelDiffModel 无需翻转，单测保持全绿）
- gen_office_world 南墙尺寸修正（原 15.4 偏移产生负尺寸 box 与 0.2m 残片），重新生成 office.sdf
- run_eval.sh：全量清杀遗留进程（run_slam_online/leg_wheel_odom/记录器/gzserver 等）、
  每次运行唯一输出目录（scene_version_ts）、记录 /degeneracy_status、leg 节点参数化
- record_gt.py：/model_states 用 RELIABLE QoS（原 best_effort 静默收不到，GT 记录实际为空）、
  /clock 深度 2000、严格递增时间戳；record_lio.py 严格递增
- evo_eval.sh 按运行目录评测；teleop corridor 模式按实测速度重设（每腿 14s×0.5 ≈ 12.7m < 15m）
- leg_wheel_odom 轮半径标定 0.05 → 0.091（仿真碰撞半径；RTF≈0.83 下墙钟测速会低估）

File: sim_ws/src/m20_description/urdf/m20.urdf (robot description, URDF)
Before this commit: robot M20, 17 links, 16 joints
Joints:
- joint fl_wheel_joint: axis 0 -1 0 -> 0 1 0
- joint fr_wheel_joint: axis 0 -1 0 -> 0 1 0
- joint hl_wheel_joint: axis 0 -1 0 -> 0 1 0
- joint hr_wheel_joint: axis 0 -1 0 -> 0 1 0
